Commit message: Camera Orientation fixed for RTB. Added Depth.

File: src/master_panda/urdf/panda.urdf.xacro (robot description, xacro)
@@ -435,31 +435,33 @@
         </inertial>
     </xacro:macro>
-    <xacro:property name="camera_length" value="0.005" />
-    <xacro:property name="camera_width" value="0.005" />
-    <xacro:property name="camera_height" value="0.002" />
+    <!-- RealSense Camera -->
     <link name="camera_link">
         <visual>
-            <geometry>
-                <box size="${camera_length} ${camera_width} ${camera_height}" />
-            </geometry>
-            <material name="Gazebo/Black">
-                <color rgba="0.5 0.5 0.5 1.0"/>
+            <origin xyz="0 0 0" rpy="0 0 0"/>
+            <geometry>
+                <box size="0.02505 0.09 0.025"/>
+            </geometry>
+            <material name="Gazebo/Blue">
+                <color rgba="0 0 1 1"/>
             </material>
         </visual>
         <collision>
-            <geometry>
-                <box size="${camera_length} ${camera_width/2} ${camera_height*2}" />
-            </geometry>
-        </collision>
-        <xacro:box_inertia m="0.1" l="${camera_length}" w="${camera_width}" h="${camera_height}"
-                           xyz="0 0 0" rpy="0 0 0" />
+            <origin xyz="0 0 0" rpy="0 0 0"/>
+            <geometry>
+                <box size="0.02505 0.09 0.025"/>
+            </geometry>
+        </collision>
+        <inertial>
+            <mass value="0.1"/>
+            <origin xyz="0 0 0" rpy="0 0 0"/>
+            <inertia ixx="0.0001" ixy="0" ixz="0" iyy="0.0001" iyz="0" izz="0.0001"/>
+        </inertial>
     </link>
     <joint name="base_camera_joint" type="fixed">
-        <parent link="panda_hand" />
-        <child link="camera_link" />
-        <origin xyz="0.02 0 0.06" rpy="0 ${-pi/2} 0" />
-    </joint>
-    <link name="camera_link_optical">
-    </link>
+        <parent link="panda_hand"/>
+        <child link="camera_link"/>
+        <origin xyz="0.02 0 0.06" rpy="0 ${-pi/2} 0"/>
+    </joint>
+    <link name="camera_link_optical"/>
     <joint name="camera_optical_joint" type="fixed">
         <origin xyz="0 0 0" rpy="${-pi/2} 0 ${-pi/2}"/>
@@ -468,11 +470,28 @@
     </joint>
     <gazebo reference="camera_link">
-        <material>Gazebo/Red</material>
-        <sensor name="camera_sensor" type="camera">
-            <pose>0 0 0.5 0 0 0</pose>
-            <visualize>true</visualize>
-            <update_rate>10.0</update_rate>
+        <material>Gazebo/Blue</material>
+        <sensor name="camera_sensor" type="depth">
+            <update_rate>30.0</update_rate>
+            <camera name="camera">
+                <horizontal_fov>1.0472</horizontal_fov>
+                <image>
+                    <width>640</width>
+                    <height>480</height>
+                    <format>R8G8B8</format>
+                </image>
+                <clip>
+                    <near>0.1</near>
+                    <far>100</far>
+                </clip>
+                <noise>
+                    <type>gaussian</type>
+                    <mean>0.0</mean>
+                    <stddev>0.007</stddev>
+                </noise>
+            </camera>
             <plugin name="camera_controller" filename="libgazebo_ros_camera.so">
                 <frame_name>camera_link_optical</frame_name>
+                <min_depth>0.1</min_depth>
+                <max_depth>100.0</max_depth>
             </plugin>
         </sensor>
