Commit message: Hard Coded Pick and Place Application

File: src/manipulator_moveit_config/config/manipulator.ros2_control.xacro (robot description, xacro)
@@ -1,16 +1,10 @@
 <?xml version="1.0"?>
 <robot xmlns:xacro="http://www.ros.org/wiki/xacro">
-    <xacro:macro name="manipulator_ros2_control" params="name initial_positions_file ros2_control_hardware_type">
-        <xacro:property name="initial_positions" value="${xacro.load_yaml(initial_positions_file)['initial_positions']}"/>
+    <xacro:macro name="manipulator_ros2_control" params="name initial_positions_file">
+        <xacro:property name="initial_positions" value="${load_yaml(initial_positions_file)['initial_positions']}"/>
         <ros2_control name="${name}" type="system">
             <hardware>
-                <xacro:if value="${ros2_control_hardware_type == 'mock_components'}">
-                    <plugin>mock_components/GenericSystem</plugin>
-                </xacro:if>
-                <xacro:if value="${ros2_control_hardware_type == 'isaac'}">
-                    <plugin>topic_based_ros2_control/TopicBasedSystem</plugin>
-                    <param name="joint_commands_topic">/isaac_joint_commands</param>
-                    <param name="joint_states_topic">/isaac_joint_states</param>
-                </xacro:if>
+                <!-- By default, set up controllers for simulation. This won't work on real hardware -->
+                <plugin>mock_components/GenericSystem</plugin>
             </hardware>
             <joint name="manipulator_joint1">
@@ -19,7 +13,5 @@
                   <param name="initial_value">${initial_positions['manipulator_joint1']}</param>
                 </state_interface>
-                <state_interface name="velocity">
-                  <param name="initial_value">0.0</param>
-                </state_interface>
+                <state_interface name="velocity"/>
             </joint>
             <joint name="manipulator_joint2">
@@ -28,7 +20,5 @@
                   <param name="initial_value">${initial_positions['manipulator_joint2']}</param>
                 </state_interface>
-                <state_interface name="velocity">
-                  <param name="initial_value">0.0</param>
-                </state_interface>
+                <state_interface name="velocity"/>
             </joint>
             <joint name="manipulator_joint3">
@@ -37,7 +27,5 @@
                   <param name="initial_value">${initial_positions['manipulator_joint3']}</param>
                 </state_interface>
-                <state_interface name="velocity">
-                  <param name="initial_value">0.0</param>
-                </state_interface>
+                <state_interface name="velocity"/>
             </joint>
             <joint name="manipulator_joint4">
@@ -46,7 +34,5 @@
                   <param name="initial_value">${initial_positions['manipulator_joint4']}</param>
                 </state_interface>
-                <state_interface name="velocity">
-                  <param name="initial_value">0.0</param>
-                </state_interface>
+                <state_interface name="velocity"/>
             </joint>
             <joint name="manipulator_joint5">
@@ -55,7 +41,5 @@
                   <param name="initial_value">${initial_positions['manipulator_joint5']}</param>
                 </state_interface>
-                <state_interface name="velocity">
-                  <param name="initial_value">0.0</param>
-                </state_interface>
+                <state_interface name="velocity"/>
             </joint>
             <joint name="manipulator_joint6">
@@ -64,7 +48,5 @@
                   <param name="initial_value">${initial_positions['manipulator_joint6']}</param>
                 </state_interface>
-                <state_interface name="velocity">
-                  <param name="initial_value">0.0</param>
-                </state_interface>
+                <state_interface name="velocity"/>
             </joint>
             <joint name="manipulator_joint7">
@@ -73,7 +55,12 @@
                   <param name="initial_value">${initial_positions['manipulator_joint7']}</param>
                 </state_interface>
-                <state_interface name="velocity">
-                  <param name="initial_value">0.0</param>
+                <state_interface name="velocity"/>
+            </joint>
+            <joint name="manipulator_finger_joint1">
+                <command_interface name="position"/>
+                <state_interface name="position">
+                  <param name="initial_value">${initial_positions['manipulator_finger_joint1']}</param>
                 </state_interface>
+                <state_interface name="velocity"/>
             </joint>
         </ros2_control>

File: src/manipulator_moveit_config/config/manipulator.urdf (robot description, URDF)
Before this commit: robot manipulator, 12 links, 11 joints
Links:
- added link manipulator_hand_sc
- added link manipulator_hand_tcp
- added link manipulator_link0_sc
- added link manipulator_link1_sc
- added link manipulator_link2_sc
- added link manipulator_link3_sc
- added link manipulator_link4_sc
- added link manipulator_link5_sc
- added link manipulator_link6_sc
- added link manipulator_link7_sc
- added link world
- link manipulator_hand: mass None -> 0.73; geometry collision mesh filename=file://$(find manipulator)/meshes/collision/hand.stl; visual mesh filename=file://$(find manipulator)/meshes/visual/hand.dae
- link manipulator_leftfinger: mass None -> 0.015; geometry collision box size=17.5e-3 15.2e-3 18.5e-3; collision box size=17.5e-3 7e-3 23.5e-3
- link manipulator_link0: mass None -> 0.629769; geometry collision mesh filename=file://$(find manipulator)/meshes/collision/link0.stl; visual mesh filename=file://$(find manipulator)/meshes/visual/link0.dae
- link manipulator_link1: mass None -> 4.970684; geometry collision mesh filename=file://$(find manipulator)/meshes/collision/link1.stl; visual mesh filename=file://$(find manipulator)/meshes/visual/link1.dae
- link manipulator_link2: mass None -> 0.646926; geometry collision mesh filename=file://$(find manipulator)/meshes/collision/link2.stl; visual mesh filename=file://$(find manipulator)/meshes/visual/link2.dae
- link manipulator_link3: mass None -> 3.228604; geometry collision mesh filename=file://$(find manipulator)/meshes/collision/link3.stl; visual mesh filename=file://$(find manipulator)/meshes/visual/link3.dae
- link manipulator_link4: mass None -> 3.587895; geometry collision mesh filename=file://$(find manipulator)/meshes/collision/link4.stl; visual mesh filename=file://$(find manipulator)/meshes/visual/link4.dae
- link manipulator_link5: mass None -> 1.225946; geometry collision mesh filename=file://$(find manipulator)/meshes/collision/link5.stl; visual mesh filename=file://$(find manipulator)/meshes/visual/link5.dae
- link manipulator_link6: mass None -> 1.47; geometry collision mesh filename=file://$(find manipulator)/meshes/collision/link6.stl; visual mesh filename=file://$(find manipulator)/meshes/visual/link6.dae
- link manipulator_link7: mass None -> 0.45; geometry collision mesh filename=file://$(find manipulator)/meshes/collision/link7.stl; visual mesh filename=file://$(find manipulator)/meshes/visual/link7.dae
- link manipulator_rightfinger: mass None -> 0.015; geometry collision box size=17.5e-3 15.2e-3 18.5e-3; collision box size=17.5e-3 7e-3 23.5e-3
Joints:
- added joint manipulator_hand_sc_joint: type fixed, parent manipulator_hand, child manipulator_hand_sc, origin rpy=0.0 0.0 0.0
- added joint manipulator_hand_tcp_joint: type fixed, parent manipulator_hand, child manipulator_hand_tcp, origin xyz=0.0 0.0 0.1034 rpy=0.0 0.0 0.0
- added joint manipulator_link0_sc_joint: type fixed, parent manipulator_link0, child manipulator_link0_sc, origin rpy=0.0 0.0 0.0
- added joint manipulator_link1_sc_joint: type fixed, parent manipulator_link1, child manipulator_link1_sc, origin rpy=0.0 0.0 0.0
- added joint manipulator_link2_sc_joint: type fixed, parent manipulator_link2, child manipulator_link2_sc, origin rpy=0.0 0.0 0.0
- added joint manipulator_link3_sc_joint: type fixed, parent manipulator_link3, child manipulator_link3_sc, origin rpy=0.0 0.0 0.0
- added joint manipulator_link4_sc_joint: type fixed, parent manipulator_link4, child manipulator_link4_sc, origin rpy=0.0 0.0 0.0
- added joint manipulator_link5_sc_joint: type fixed, parent manipulator_link5, child manipulator_link5_sc, origin rpy=0.0 0.0 0.0
- added joint manipulator_link6_sc_joint: type fixed, parent manipulator_link6, child manipulator_link6_sc, origin rpy=0.0 0.0 0.0
- added joint manipulator_link7_sc_joint: type fixed, parent manipulator_link7, child manipulator_link7_sc, origin rpy=0.0 0.0 0.0
- added joint world_joint: type fixed, parent world, child manipulator_link0, origin xyz=0.0 0.0 0.0 rpy=0.0 0.0 0.0
- joint manipulator_finger_joint1: limit lower=0.0 upper=0.04 effort=20 velocity=0.2 -> lower=0.0 upper=0.04 effort=20.0 velocity=0.2
- joint manipulator_finger_joint2: limit lower=0.0 upper=0.04 effort=20 velocity=0.2 -> lower=0.0 upper=0.04 effort=20.0 velocity=0.2
- joint manipulator_joint8: axis 0 0 0 -> (none)
