Commit message: Hard Coded Pick and Place Application

File: src/manipulator_moveit_config/config/manipulator.urdf.xacro (robot description, xacro)
@@ -1,19 +1,3 @@
 <?xml version="1.0"?>
-<!-- =================================================================================== -->
-<!-- |    This document was autogenerated by xacro from /opt/ros/kinetic/share/moveit_resources/manipulator_description/urdf/manipulator.urdf | -->
-<!-- |    EDITING THIS FILE BY HAND IS NOT RECOMMENDED                                 | -->
-<!-- =================================================================================== -->
-<!-- <?xml version="1.0"?> -->
-<!-- <robot xmlns:xacro="http://www.ros.org/wiki/xacro" name="manipulator"> -->
-    <!-- <xacro:arg name="initial_positions_file" default="initial_positions.yaml" /> -->
-    <!-- <xacro:arg name="ros2_control_hardware_type" default="mock_components" /> -->
-    <!-- Import panda urdf file -->
-    <!-- <xacro:include filename="$(find manipulator_moveit_config)/config/manipulator.urdf" /> -->
-    <!-- Import panda ros2_control description -->
-    <!-- <xacro:include filename="manipulator.ros2_control.xacro" /> -->
-    <!-- <xacro:include filename="manipulator_hand.ros2_control.xacro" /> -->
-    <!-- <xacro:manipulator_ros2_control name="ManipulatorFakeSystem" initial_positions_file="$(arg initial_positions_file)" ros2_control_hardware_type="$(arg ros2_control_hardware_type)"/> -->
-    <!-- <xacro:manipulator_hand_ros2_control name="ManipulatorHandFakeSystem" ros2_control_hardware_type="$(arg ros2_control_hardware_type)"/> -->
-<!-- </robot>  -->
 <robot name="manipulator" xmlns:xacro="http://www.ros.org/wiki/xacro">
     <link name="manipulator_link0">
@@ -34,8 +18,6 @@
         </inertial>
     </link>
-    <!-- sub-link defining coarse geometries of real robot's internal self-collision -->
     <link name="manipulator_link0_sc">
     </link>
-    <!-- fixed joint between both sub-links -->
     <joint name="manipulator_link0_sc_joint" type="fixed">
         <origin rpy="0.0 0.0 0.0"/>
@@ -60,8 +42,6 @@
         </inertial>
     </link>
-    <!-- sub-link defining coarse geometries of real robot's internal self-collision -->
     <link name="manipulator_link1_sc">
     </link>
-    <!-- fixed joint between both sub-links -->
     <joint name="manipulator_link1_sc_joint" type="fixed">
         <origin rpy="0.0 0.0 0.0"/>
@@ -95,8 +75,6 @@
         </inertial>
     </link>
-    <!-- sub-link defining coarse geometries of real robot's internal self-collision -->
     <link name="manipulator_link2_sc">
     </link>
-    <!-- fixed joint between both sub-links -->
     <joint name="manipulator_link2_sc_joint" type="fixed">
         <origin rpy="0.0 0.0 0.0"/>
@@ -130,8 +108,6 @@
         </inertial>
     </link>
-    <!-- sub-link defining coarse geometries of real robot's internal self-collision -->
     <link name="manipulator_link3_sc">
     </link>
-    <!-- fixed joint between both sub-links -->
     <joint name="manipulator_link3_sc_joint" type="fixed">
         <origin rpy="0.0 0.0 0.0"/>
@@ -165,8 +141,6 @@
         </inertial>
     </link>
-    <!-- sub-link defining coarse geometries of real robot's internal self-collision -->
     <link name="manipulator_link4_sc">
     </link>
-    <!-- fixed joint between both sub-links -->
     <joint name="manipulator_link4_sc_joint" type="fixed">
         <origin rpy="0.0 0.0 0.0"/>
@@ -180,5 +154,5 @@
         <child link="manipulator_link4" />
         <axis xyz="0 0 1" />
-        <limit effort="87" lower="-3.1416" upper="0.0873" velocity="2.3925" />
+        <limit effort="87" lower="-3.1416" upper="0.088" velocity="2.3925" />
         <dynamics D="1.0" K="7000.0" damping="0.003" friction="0.0" mu_coulomb="0.0" mu_viscous="16.0"/>
     </joint>
@@ -200,8 +174,6 @@
         </inertial>
     </link>
-    <!-- sub-link defining coarse geometries of real robot's internal self-collision -->
     <link name="manipulator_link5_sc">
     </link>
-    <!-- fixed joint between both sub-links -->
     <joint name="manipulator_link5_sc_joint" type="fixed">
         <origin rpy="0.0 0.0 0.0"/>
@@ -235,8 +207,6 @@
         </inertial>
     </link>
-    <!-- sub-link defining coarse geometries of real robot's internal self-collision -->
     <link name="manipulator_link6_sc">
     </link>
-    <!-- fixed joint between both sub-links -->
     <joint name="manipulator_link6_sc_joint" type="fixed">
         <origin rpy="0.0 0.0 0.0"/>
@@ -246,5 +216,5 @@
     <joint name="manipulator_joint6" type="revolute">
         <safety_controller k_position="100.0" k_velocity="40.0" soft_lower_limit="-0.0175" soft_upper_limit="3.7525" />
-        <origin rpy="1.57079632679 0 0" xyz="0 0 0" />
+        <origin rpy="0.9 0 0" xyz="0 0 0" /> <!--1.57079632679-->
         <parent link="manipulator_link5" />
         <child link="manipulator_link6" />
@@ -270,8 +240,6 @@
         </inertial>
     </link>
-    <!-- sub-link defining coarse geometries of real robot's internal self-collision -->
     <link name="manipulator_link7_sc">
     </link>
-    <!-- fixed joint between both sub-links -->
     <joint name="manipulator_link7_sc_joint" type="fixed">
         <origin rpy="0.0 0.0 0.0"/>
@@ -293,5 +261,5 @@
         <parent link="manipulator_link7" />
         <child link="manipulator_link8" />
-        <!-- <axis xyz="0 0 0" /> -->
+        <axis xyz="0 0 0" />
     </joint>
     <joint name="manipulator_hand_joint" type="fixed">
@@ -317,8 +285,6 @@
         </inertial>
     </link>
-    <!-- sub-link defining coarse geometries of real robot's internal self-collision -->
-    <link name="manipulator_hand_sc">
-    </link>
-    <!-- fixed joint between both sub-links -->
+    <!-- <link name="manipulator_hand_sc">
+    </link>
     <joint name="manipulator_hand_sc_joint" type="fixed">
         <origin rpy="0.0 0.0 0.0"/>
@@ -326,5 +292,4 @@
         <child link="manipulator_hand_sc"/>
     </joint>
-    <!-- Define the hand_tcp frame -->
     <link name="manipulator_hand_tcp"/>
     <joint name="manipulator_hand_tcp_joint" type="fixed">
@@ -332,5 +297,5 @@
         <parent link="manipulator_hand"/>
         <child link="manipulator_hand_tcp"/>
-    </joint>
+    </joint> -->
     <link name="manipulator_leftfinger">
         <visual>
@@ -339,5 +304,4 @@
             </geometry>
         </visual>
-        <!-- screw mount -->
         <collision>
             <origin rpy="0.0 0.0 0.0" xyz="0.0 18.5e-3 11.0e-3"/>
@@ -346,5 +310,4 @@
             </geometry>
         </collision>
-        <!-- cartriage sledge -->
         <collision>
         <origin rpy="0.0 0.0 0.0" xyz="0.0 6.8e-3 2.2e-3"/>
@@ -353,5 +316,4 @@
         </geometry>
         </collision>
-        <!-- diagonal finger -->
         <collision>
         <origin rpy="0.5235987755982988 0.0 0.0" xyz="0.0 15.9e-3 28.35e-3"/>
@@ -360,5 +322,4 @@
         </geometry>
         </collision>
-        <!-- rubber tip with which to grasp -->
         <collision>
         <origin rpy="0.0 0.0 0.0" xyz="0 7.58e-3 45.25e-3"/>
@@ -380,5 +341,4 @@
             </geometry>
         </visual>
-         <!-- screw mount -->
         <collision>
         <origin rpy="0.0 0.0 0.0" xyz="0.0 -18.5e-3 11e-3"/>
@@ -387,5 +347,4 @@
         </geometry>
         </collision>
-        <!-- cartriage sledge -->
         <collision>
         <origin rpy="0.0 0.0 0.0" xyz="0.0 -6.8e-3 2.2e-3"/>
@@ -394,5 +353,4 @@
         </geometry>
         </collision>
-        <!-- diagonal finger -->
         <collision>
         <origin rpy="-0.5235987755982988 0.0 0.0" xyz="0 -15.9e-3 28.35e-3"/>
@@ -401,5 +359,4 @@
         </geometry>
         </collision>
-        <!-- rubber tip with which to grasp -->
         <collision>
         <origin rpy="0.0 0.0 0.0" xyz="0.0 -7.58e-3 45.25e-3"/>
@@ -419,6 +376,6 @@
         <origin rpy="0 0 0" xyz="0 0 0.0584" />
         <axis xyz="0 1 0" />
-        <limit effort="100.0" lower="0.0" upper="0.04" velocity="0.2" />
-        <dynamics damping="0.3"/>
+        <limit effort="20.0" lower="0.0" upper="0.04" velocity="0.2" />
+        <dynamics damping="0.3" friction="0"/>
     </joint>
     <joint name="manipulator_finger_joint2" type="prismatic">
@@ -427,7 +384,7 @@
         <origin rpy="0 0 0" xyz="0 0 0.0584" />
         <axis xyz="0 -1 0" />
-        <limit effort="100.0" lower="0.0" upper="0.04" velocity="0.2" />
-        <mimic joint="manipulator_finger_joint1" />
-        <dynamics damping="0.3"/>
+        <limit effort="20.0" lower="0.0" upper="0.04" velocity="0.2" />
+        <mimic joint="manipulator_finger_joint1"/>
+        <dynamics damping="0.3"  friction="0"/>
     </joint>
     <link name="world">
@@ -438,5 +395,5 @@
         <child link="manipulator_link0"/>
     </joint>
-    <xacro:macro name="box_inertia" params="m l w h xyz rpy">
+    <!-- <xacro:macro name="box_inertia" params="m l w h xyz rpy">
         <inertial>
             <origin xyz="${xyz}" rpy="${rpy}" />
@@ -446,7 +403,6 @@
                      izz="${(m/12) * (w*w + h*h)}" />
         </inertial>
-    </xacro:macro>
-    <!-- RealSense Camera -->
-    <link name="camera_link">
+    </xacro:macro> -->
+    <!-- <link name="camera_link">
         <visual>
             <origin xyz="0 0 0" rpy="0 0 0"/>
@@ -509,81 +465,92 @@
         </sensor>
     </gazebo>
+     -->
     <ros2_control name="GazeboSystem" type="system">
         <hardware>
             <plugin>gazebo_ros2_control/GazeboSystem</plugin>
         </hardware>
-        <!-- Arm joints -->
         <joint name="manipulator_joint1">
-            <param name="initial_position">0.0</param>
-            <command_interface name="effort"/>
-            <command_interface name="velocity"/>
-            <command_interface name="position"/>
-            <state_interface name="position"/>
+            <command_interface name="effort"/>
+            <command_interface name="velocity"/>
+            <command_interface name="position"/>
+            <state_interface name="position">
+                <param name="initial_value">0.0</param>
+            </state_interface>
             <state_interface name="velocity"/>
             <state_interface name="effort"/>
         </joint>
         <joint name="manipulator_joint2">
-            <param name="initial_position">-0.785</param>
-            <command_interface name="effort"/>
-            <command_interface name="velocity"/>
-            <command_interface name="position"/>
-            <state_interface name="position"/>
+            <command_interface name="effort"/>
+            <command_interface name="velocity"/>
+            <command_interface name="position"/>
+            <state_interface name="position">
+                <param name="initial_value">-0.785</param>
+            </state_interface>
             <state_interface name="velocity"/>
             <state_interface name="effort"/>
         </joint>
         <joint name="manipulator_joint3">
-            <param name="initial_position">0.0</param>
-            <command_interface name="effort"/>
-            <command_interface name="velocity"/>
-            <command_interface name="position"/>
-            <state_interface name="position"/>
+            <command_interface name="effort"/>
+            <command_interface name="velocity"/>
+            <command_interface name="position"/>
+            <state_interface name="position">
+                <param name="initial_value">0.3</param>
+            </state_interface>
             <state_interface name="velocity"/>
             <state_interface name="effort"/>
         </joint>
         <joint name="manipulator_joint4">
-            <param name="initial_position">-2.356</param>
-            <command_interface name="effort"/>
-            <command_interface name="velocity"/>
-            <command_interface name="position"/>
-            <state_interface name="position"/>
+            <command_interface name="effort"/>
+            <command_interface name="velocity"/>
+            <command_interface name="position"/>
+            <state_interface name="position">
+                <param name="initial_value">-2.356</param>
+            </state_interface>
             <state_interface name="velocity"/>
             <state_interface name="effort"/>
         </joint>
         <joint name="manipulator_joint5">
-            <param name="initial_position">0.0</param>
-            <command_interface name="effort"/>
-            <command_interface name="velocity"/>
-            <command_interface name="position"/>
-            <state_interface name="position"/>
+            <command_interface name="effort"/>
+            <command_interface name="velocity"/>
+            <command_interface name="position"/>
+            <state_interface name="position">
+                <param name="initial_value">0.0</param>
+            </state_interface>
             <state_interface name="velocity"/>
             <state_interface name="effort"/>
         </joint>
         <joint name="manipulator_joint6">
-            <param name="initial_position">1.571</param>
-            <command_interface name="effort"/>
-            <command_interface name="velocity"/>
-            <command_interface name="position"/>
-            <state_interface name="position"/>
+            <command_interface name="effort"/>
+            <command_interface name="velocity"/>
+            <command_interface name="position"/>
+            <state_interface name="position">
+                <param name="initial_value">1.571</param>
+            </state_interface>
             <state_interface name="velocity"/>
             <state_interface name="effort"/>
         </joint>
         <joint name="manipulator_joint7">
-            <param name="initial_position">0.785</param>
-            <command_interface name="effort"/>
-            <command_interface name="velocity"/>
-            <command_interface name="position"/>
-            <state_interface name="position"/>
-            <state_interface name="velocity"/>
-            <state_interface name="effort"/>
-        </joint>
-        <!-- Gripper joint -->
+            <command_interface name="effort"/>
+            <command_interface name="velocity"/>
+            <command_interface name="position"/>
+            <state_interface name="position">
+                <param name="initial_value">0.785</param>
+            </state_interface>
+            <state_interface name="velocity"/>
+            <state_interface name="effort"/>
+        </joint>
         <joint name="manipulator_finger_joint1">
-            <param name="initial_position">1.0</param>
-            <command_interface name="effort"/>
-            <command_interface name="velocity"/>
-            <command_interface name="position"/>
-            <state_interface name="position"/>
-            <state_interface name="velocity"/>
-            <state_interface name="effort"/>
+            <command_interface name="effort"/>
+            <command_interface name="velocity"/>
+            <command_interface name="position"/>
+            <state_interface name="position">
+                <param name="initial_position">0.0</param>
+            </state_interface>
+            <state_interface name="velocity"/>
+            <state_interface name="effort"/>
+        </joint>
+        <joint name="manipulator_finger_joint2">
+            <param name="mimic">manipulator_finger_joint1</param>
+            <param name="multiplier">1</param>
         </joint>
     </ros2_control>
@@ -592,8 +559,7 @@
             <robot_param>robot_description</robot_param>
             <robot_param_node>robot_state_publisher</robot_param_node>
-            <parameters>/home/humble/Projects/pick_place/src/manipulator/config/controllers.yaml</parameters>
+            <parameters>$(find manipulator)/config/controllers.yaml</parameters>
         </plugin>
     </gazebo>
-    <!-- Add Gazebo materials for each link -->
     <gazebo reference="manipulator_link0">
         <material>Gazebo/Grey</material>
@@ -629,3 +595,7 @@
         <material>Gazebo/Grey</material>
     </gazebo>
+    <gazebo>
+        <plugin name="gazebo_link_attacher" filename="libgazebo_link_attacher.so">
+        </plugin>
+    </gazebo>
 </robot>

File: src/manipulator_moveit_config/config/square_red.urdf.xacro (robot description, xacro)
@@ -2,5 +2,5 @@
 <sdf version="1.6">
     <model name="square_object">
-        <static>true</static>
+        <static>false</static>
         <link name="square_object_link">
             <pose>0 0 0 0 0 0</pose>
@@ -8,10 +8,10 @@
                 <geometry>
                     <box>
-                        <size>0.04 0.04 0.04</size>
+                        <size>0.025 0.025 0.1</size>
                     </box>
                 </geometry>
                 <material>
-                    <ambient>0 0 1 1</ambient>
-                    <diffuse>0 0 1 1</diffuse>
+                    <ambient>1 0 0 1</ambient>
+                    <diffuse>1 0 0 1</diffuse>
                 </material>
             </visual>
@@ -19,16 +19,8 @@
                 <geometry>
                     <box>
-                        <size>0.01 0.01 0.01</size>
+                        <size>0.025 0.025 0.1</size>
                     </box>
                 </geometry>
             </collision>
-            <inertial>
-                <mass>0.1</mass>
-                <inertia>
-                    <ixx>0.0001</ixx>
-                    <iyy>0.0001</iyy>
-                    <izz>0.0001</izz>
-                </inertia>
-            </inertial>
         </link>
     </model>
